File: PCB/stylophone/pomiary.sch (EAGLE design)
At the start: 27 parts, among them IC2 LM358N, X1 332-02

Commit message: vibrato freq
Parts:
- removed NA4, NA4#, NB4, NC4, NC4#, ND4, ND4#, NE4, NF4, NF4#, NG4, NG4#: (no value), resistor:R-EU_M1206
- removed SP1: AL60P, buzzer:AL60P
- removed X1: 332-02, con-garry:332-02
- added SV2: (no value), con-lstb:MA04-1
- added U$1: ZASILACZ, Przyrzady pomiarowe:ZASILACZ
- added U$2, U$3, U$4: OSCYLOSKOP_AC_AC, Przyrzady pomiarowe:OSCYLOSKOP_AC_AC
- R2: device resistor:R-EU_0204/7 -> resistor:R-EU_M1206
Connections:
- net GND: now also SV2.2, SV2.4, U$1.CH1-, U$2.GND, U$3.GND, U$4.GND; no longer SP1.2, TONE.GND, X1-1.S
- net N$5: now also U$3.CH1
- net NOTE: no longer NA4#.2, NA4.2, NB4.2, NC4#.2, NC4.2, ND4#.2, ND4.2, NE4.2, NF4#.2, NF4.2, NG4#.2, NG4.2
- net NOTSTYLUS: now also U$2.CH1
- net OUTPUT: now also SV2.3, U$3.CH2; no longer SP1.1
- net STYLUS: now also U$4.CH1
- net TONE: now also U$4.CH2
- net VCC: now also SV2.1, U$1.CH1+; no longer X1-2.S
- net VIBRATO: now also U$2.CH2
Other:
- moved on the sheet: C2, C3, C4, C5, IC2A, R2, R3, R4, R5, R6, R7, TONE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
