File: PCB/stylophone/stylophone.brd (EAGLE design)
At the start: 102.5 x 80 mm, 27 parts, among them IC2 LM358N, X1 332-02

Commit message: vibrato freq
Parts:
- removed SP1: AL60P, buzzer:AL60P
- removed X1: 332-02, con-garry:332-02
- added SV1: (no value), con-lstb:MA04-1
Connections:
- net GND: now also SV1.2, SV1.4; no longer SP1.2, X1.1
- net OUTPUT: now also SV1.3; no longer SP1.1
- net VCC: now also SV1.1; no longer X1.2
Routing:
- net NOTE: track 98.0 -> 40.7 mm
- net VCC: track 91.5 -> 87.4 mm
- net OUTPUT: track 11.7 -> 8.18 mm
- net GND: track 157.3 -> 155.8 mm
Changed lines of the file:
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@@
 <element name="NA4#" library="resistor" package="M1206" value="" x="57.15" y="8.89" rot="R90"/>
 <element name="NB4" library="resistor" package="M1206" value="" x="62.23" y="8.89" rot="R90"/>
-<element name="SP1" library="buzzer" package="AL60P" value="AL60P" x="21.59" y="26.67" rot="R270">
-<attribute name="OC_NEWARK" value="unknown" x="21.59" y="26.67" size="1.778" layer="27" rot="R270" display="off"/>
-<attribute name="MPN" value="" x="21.59" y="26.67" size="1.778" layer="27" rot="R270" display="off"/>
-<attribute name="MF" value="" x="21.59" y="26.67" size="1.778" layer="27" rot="R270" display="off"/>
-<attribute name="OC_FARNELL" value="unknown" x="21.59" y="26.67" size="1.778" layer="27" rot="R270" display="off"/>
+<element name="SV1" library="con-lstb" package="MA04-1" value="" x="1.27" y="-3.81">
+<attribute name="OC_NEWARK" value="unknown" x="1.27" y="-3.81" size="1.778" layer="27" display="off"/>
+<attribute name="MPN" value="" x="1.27" y="-3.81" size="1.778" layer="27" display="off"/>
+<attribute name="MF" value="" x="1.27" y="-3.81" size="1.778" layer="27" display="off"/>
+<attribute name="OC_FARNELL" value="unknown" x="1.27" y="-3.81" size="1.778" layer="27" display="off"/>
 </element>
-<element name="X1" library="con-garry" package="332-02" value="332-02" x="0" y="25.4" rot="R180"/>
 </elements>
 <signals>
@@
 <wire x1="24.13" y1="44.45" x2="26.67" y2="44.45" width="1.016" layer="1"/>
 <contactref element="IC2" pad="8"/>
-<contactref element="X1" pad="2"/>
-<wire x1="0" y1="24.4" x2="0" y2="20.32" width="1.016" layer="1"/>
 <wire x1="0" y1="20.32" x2="1.27" y2="19.05" width="1.016" layer="1"/>
 <wire x1="1.27" y1="19.05" x2="11.43" y2="19.05" width="1.016" layer="1"/>
@@
 <wire x1="27.94" y1="27.94" x2="27.94" y2="21.59" width="1.016" layer="1"/>
 <wire x1="27.94" y1="21.59" x2="25.4" y2="19.05" width="1.016" layer="1"/>
+<contactref element="SV1" pad="1"/>
 <wire x1="27.94" y1="27.94" x2="38.1" y2="26.54" width="0" layer="19" extent="1-1"/>
+<wire x1="-2.54" y1="-3.81" x2="1.27" y2="19.05" width="0" layer="19" extent="1-1"/>
 </signal>
 <signal name="OUTPUT">
 <contactref element="IC2" pad="2"/>
 <contactref element="IC2" pad="1"/>
-<contactref element="SP1" pad="1"/>
-<wire x1="10.16" y1="29.21" x2="12.7" y2="29.21" width="0.4064" layer="1"/>
+<contactref element="SV1" pad="3"/>
 <wire x1="12.7" y1="29.21" x2="20.8788" y2="29.21" width="0.4064" layer="1"/>
-<wire x1="20.8788" y1="29.21" x2="21.59" y2="29.9212" width="0.4064" layer="1"/>
+<wire x1="10.16" y1="29.21" x2="12.7" y2="29.21" width="0" layer="19" extent="1-1"/>
+<wire x1="2.54" y1="-3.81" x2="10.16" y2="29.21" width="0" layer="19" extent="1-1"/>
 </signal>
 <signal name="N$5">
@@
 <wire x1="5.08" y1="46.99" x2="7.62" y2="49.53" width="1.016" layer="1"/>
 <wire x1="5.08" y1="29.21" x2="5.08" y2="46.99" width="1.016" layer="1"/>
-<contactref element="X1" pad="1"/>
-<contactref element="SP1" pad="2"/>
-<wire x1="0" y1="26.4" x2="0" y2="27.94" width="1.016" layer="1"/>
 <wire x1="0" y1="27.94" x2="1.27" y2="29.21" width="1.016" layer="1"/>
 <wire x1="1.27" y1="29.21" x2="5.08" y2="29.21" width="1.016" layer="1"/>
@@
 <wire x1="38.1" y1="34.29" x2="38.1" y2="41.91" width="1.016" layer="1"/>
 <wire x1="33.02" y1="46.99" x2="19.05" y2="46.99" width="1.016" layer="1"/>
-<wire x1="21.59" y1="22.86" x2="21.59" y2="23.4188" width="0" layer="19" extent="1-1"/>
 <wire x1="33.02" y1="46.99" x2="38.1" y2="41.91" width="1.016" layer="1"/>
+<contactref element="SV1" pad="4"/>
+<contactref element="SV1" pad="2"/>
+<wire x1="5.08" y1="-3.81" x2="6.35" y2="25.4" width="0" layer="19" extent="1-1"/>
+<wire x1="0" y1="-3.81" x2="5.08" y2="-3.81" width="0" layer="19" extent="1-1"/>
 </signal>
 <signal name="TONE">
@@
 <signal name="NOTE">
 <contactref element="R2" pad="2"/>
-<contactref element="TONE" pad="7"/>
+<wire x1="25.4" y1="34.29" x2="24.13" y2="35.56" width="0.4064" layer="1"/>
+<wire x1="24.13" y1="35.56" x2="24.13" y2="40.64" width="0.4064" layer="1"/>
+<wire x1="25.4" y1="41.91" x2="24.13" y2="40.64" width="0.4064" layer="1"/>
+<wire x1="30.48" y1="36.7" x2="30.48" y2="35.56" width="0.4064" layer="1"/>
+<wire x1="30.48" y1="35.56" x2="30.48" y2="10.29" width="0.4064" layer="1"/>
+<wire x1="25.4" y1="34.29" x2="29.21" y2="34.29" width="0.4064" layer="1"/>
+<wire x1="29.21" y1="34.29" x2="30.48" y2="35.56" width="0.4064" layer="1"/>
 <contactref element="NB4" pad="2"/>
 <contactref element="NA4#" pad="2"/>
@@
 <contactref element="NC4#" pad="2"/>
 <contactref element="NC4" pad="2"/>
-<wire x1="6.35" y1="10.29" x2="11.43" y2="10.29" width="0.4064" layer="1"/>
-<wire x1="11.43" y1="10.29" x2="16.51" y2="10.29" width="0.4064" layer="1"/>
-<wire x1="16.51" y1="10.29" x2="21.59" y2="10.29" width="0.4064" layer="1"/>
-<wire x1="21.59" y1="10.29" x2="26.67" y2="10.29" width="0.4064" layer="1"/>
-<wire x1="26.67" y1="10.29" x2="30.48" y2="10.29" width="0.4064" layer="1"/>
-<wire x1="30.48" y1="10.29" x2="31.75" y2="10.29" width="0.4064" layer="1"/>
-<wire x1="31.75" y1="10.29" x2="36.83" y2="10.29" width="0.4064" layer="1"/>
-<wire x1="36.83" y1="10.29" x2="41.91" y2="10.29" width="0.4064" layer="1"/>
-<wire x1="41.91" y1="10.29" x2="46.99" y2="10.29" width="0.4064" layer="1"/>
-<wire x1="46.99" y1="10.29" x2="52.07" y2="10.29" width="0.4064" layer="1"/>
-<wire x1="52.07" y1="10.16" x2="52.07" y2="10.29" width="0.4064" layer="1"/>
-<wire x1="52.07" y1="10.29" x2="57.15" y2="10.29" width="0.4064" layer="1"/>
-<wire x1="57.15" y1="10.29" x2="62.23" y2="10.29" width="0.4064" layer="1"/>
-<wire x1="25.4" y1="34.29" x2="24.13" y2="35.56" width="0.4064" layer="1"/>
-<wire x1="24.13" y1="35.56" x2="24.13" y2="40.64" width="0.4064" layer="1"/>
-<wire x1="26.67" y1="41.91" x2="25.4" y2="41.91" width="0.4064" layer="1"/>
-<wire x1="25.4" y1="41.91" x2="24.13" y2="40.64" width="0.4064" layer="1"/>
-<wire x1="30.48" y1="36.7" x2="30.48" y2="35.56" width="0.4064" layer="1"/>
-<wire x1="30.48" y1="35.56" x2="30.48" y2="10.29" width="0.4064" layer="1"/>
-<wire x1="25.4" y1="34.29" x2="29.21" y2="34.29" width="0.4064" layer="1"/>
-<wire x1="29.21" y1="34.29" x2="30.48" y2="35.56" width="0.4064" layer="1"/>
+<contactref element="TONE" pad="7"/>
+<wire x1="57.15" y1="10.29" x2="62.23" y2="10.29" width="0" layer="19" extent="1-1"/>
+<wire x1="52.07" y1="10.29" x2="57.15" y2="10.29" width="0" layer="19" extent="1-1"/>
+<wire x1="46.99" y1="10.29" x2="52.07" y2="10.29" width="0" layer="19" extent="1-1"/>
+<wire x1="41.91" y1="10.29" x2="46.99" y2="10.29" width="0" layer="19" extent="1-1"/>
+<wire x1="36.83" y1="10.29" x2="41.91" y2="10.29" width="0" layer="19" extent="1-1"/>
+<wire x1="31.75" y1="10.29" x2="36.83" y2="10.29" width="0" layer="19" extent="1-1"/>
+<wire x1="30.48" y1="10.29" x2="31.75" y2="10.29" width="0" layer="19" extent="1-1"/>
+<wire x1="26.67" y1="41.91" x2="25.4" y2="41.91" width="0" layer="19" extent="1-1"/>
+<wire x1="26.67" y1="10.29" x2="30.48" y2="10.29" width="0" layer="19" extent="1-1"/>
+<wire x1="21.59" y1="10.29" x2="26.67" y2="10.29" width="0" layer="19" extent="1-1"/>
+<wire x1="16.51" y1="10.29" x2="21.59" y2="10.29" width="0" layer="19" extent="1-1"/>
+<wire x1="11.43" y1="10.29" x2="16.51" y2="10.29" width="0" layer="19" extent="1-1"/>
+<wire x1="6.35" y1="10.29" x2="11.43" y2="10.29" width="0" layer="19" extent="1-1"/>
 </signal>
 <signal name="N$1">
