File: PCB/stylophone/stylophone.sch (EAGLE design)
At the start: 27 parts, among them IC2 LM358N, X1 332-02

Commit message: vibrato freq
Parts:
- removed SP1: AL60P, buzzer:AL60P
- removed X1: 332-02, con-garry:332-02
- added SV1: (no value), con-lstb:MA04-1
Connections:
- net GND: now also SV1.2, SV1.4; no longer SP1.2, X1-1.S
- net OUTPUT: now also SV1.3; no longer SP1.1
- net VCC: now also SV1.1; no longer X1-2.S
Other:
- moved on the sheet: IC2A, NA4, NA4#, NB4, NC4, NC4#, ND4, ND4#, NE4, NF4, NF4#, NG4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
