File: PCB/stylophone.brd (EAGLE design)
At the start: 100 x 73.7 mm, 25 parts, among them IC2 LM358N

Commit message: v2
Parts:
- removed C5: 10u, capacitor-wima:C2.5-5
- added SV1: (no value), con-lstb:MA04-1
- R2: device resistor:0204/7 -> resistor:M1206
- moved R7 43.2 mm to (45.7, 21.6), turned to 0 degrees
- moved R3 42.4 mm to (38.1, 27.9), turned to 90 degrees
- moved VIBRATO 28.0 mm to (45.7, 30.5), turned to 90 degrees
- moved C4 25.4 mm to (41.9, 41.9), turned to 90 degrees
- moved R6 16.7 mm to (53.3, 33.0), turned to 270 degrees
- moved NA4 15.2 mm to (52.1, 8.89)
- moved NA4# 15.2 mm to (57.1, 8.89)
- moved NB4 15.2 mm to (62.2, 8.89)
- moved NC4 15.2 mm to (6.35, 8.89)
- moved NC4# 15.2 mm to (11.4, 8.89)
- moved ND4 15.2 mm to (16.5, 8.89)
- moved ND4# 15.2 mm to (21.6, 8.89)
- moved NE4 15.2 mm to (26.7, 8.89)
- moved NF4 15.2 mm to (31.8, 8.89)
- moved NF4# 15.2 mm to (36.8, 8.89)
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Connections:
- net GND: now also SV1.2, SV1.4; no longer C5.2
- net OUTPUT: now also SV1.3
- net VCC: now also SV1.1
- net VIBRATO: no longer C5.1
Routing:
- net NOTE: track 83.6 -> 40.7 mm
- net VCC: track 46.2 -> 87.4 mm
- net N$5: track 8.94 -> 15.3 mm
- net OUTPUT: track 2.54 -> 8.18 mm
- net STYLUS: track 3.81 -> 6.35 mm, vias 0 -> 1
- net GND: track 140.2 -> 141.8 mm
- net VIBRATO: track 8.76 -> 7.80 mm
Other:
- board size 100 x 73.7 mm -> 102.5 x 80 mm

Commit message: almost finished
Parts:
- removed R4: 100k, resistor:M1206
- removed R5: 50k, resistor:M1206
- removed R6: 1k, resistor:M1206
- removed SV1: (no value), con-lstb:MA04-1
- added R1, R8: (no value), resistor:RTRIM5X
- added SV2: (no value), con-lstb:MA05-1
- R7: device resistor:0204/7 -> resistor:M1206
- moved R3 37.7 mm to (58.4, 59.7), turned to 270 degrees
- moved R7 35.4 mm to (58.4, 54.6), turned to 270 degrees
- moved IC2 32.0 mm to (5.08, 57.1), turned to 90 degrees
- moved VIBRATO 26.9 mm to (49.5, 57.1), turned to 270 degrees
- moved C3 23.4 mm to (40.6, 59.7)
- moved NC4 22.2 mm to (17.8, 27.9)
- moved ND4# 22.2 mm to (33.0, 27.9)
- moved NG4 22.2 mm to (53.3, 27.9)
- moved NA4 22.2 mm to (63.5, 27.9)
- moved NA4# 22.2 mm to (68.6, 27.9)
- moved NB4 22.2 mm to (73.7, 27.9)
- moved NC4# 22.2 mm to (22.9, 27.9)
- moved ND4 22.2 mm to (27.9, 27.9)
- moved NE4 22.2 mm to (38.1, 27.9)
- moved NF4 22.2 mm to (43.2, 27.9)
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Connections:
- net GND: now also R1.1, R8.1, SV2.2, SV2.5; no longer R4.2, SV1.2, SV1.4
- net N$2: now also R8.3; no longer R6.2
- net N$5: now also R1.2; no longer R4.1, R5.2
- net OUTPUT: now also SV2.4; no longer SV1.3
- net STYLUS: now also SV2.3
- net TONE: now also R1.3; no longer R5.1
- net VCC: now also SV2.1; no longer SV1.1
- net VIBRATO: now also R8.2; no longer R6.1
Routing:
- net STYLUS: track 6.35 -> 33.9 mm, vias 1 -> 0
- net NOTE: track 40.7 -> 61.3 mm
- net GND: track 141.8 -> 125.7 mm
- net VIBRATO: track 7.80 -> 21.2 mm
- net N$3: track 20.0 -> 7.78 mm
- net NOTSTYLUS: track 30.6 -> 19.9 mm
- net N$5: track 15.3 -> 5.93 mm
- net N$2: track 3.86 -> 10.8 mm
- net TONE: track 8.76 -> 4.40 mm
- net VCC: track 87.4 -> 84.2 mm
- net N$9: track 0.00 -> 2.54 mm
- net N$20: track 0.00 -> 2.54 mm
- net N$19: track 0.00 -> 2.54 mm
- net N$18: track 0.00 -> 2.54 mm
- net N$17: track 0.00 -> 2.54 mm
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- added copper zone on layer 1, net N$4
- added copper zone on layer 1, net N$6
- added copper zone on layer 1, net N$7
- added copper zone on layer 1, net N$8

Commit message: almost done
Parts:
- added R4: (no value), rcl:0204/5
- moved NA4 16.7 mm to (53.5, 41.3)
- moved NA4# 16.7 mm to (58.6, 41.3)
- moved NB4 16.7 mm to (63.7, 41.3)
- moved NC4 16.7 mm to (7.78, 41.3)
- moved NC4# 16.7 mm to (12.9, 41.3)
- moved ND4 16.7 mm to (17.9, 41.3)
- moved ND4# 16.7 mm to (23.0, 41.3)
- moved NE4 16.7 mm to (28.1, 41.3)
- moved NF4 16.7 mm to (33.2, 41.3)
- moved NF4# 16.7 mm to (38.3, 41.3)
- moved NG4 16.7 mm to (43.3, 41.3)
- moved NG4# 16.7 mm to (48.4, 41.3)
- moved C3 6.32 mm to (46.6, 61.7)
- moved C4 6.32 mm to (59.3, 50.3)
- moved IC2 6.32 mm to (11.1, 59.1)
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Connections:
- new net KEYBOARD: NA4#.2, NA4.2, NB4.2, NC4#.2, NC4.2, ND4#.2, ND4.2, NE4.2, NF4#.2, NF4.2, NG4#.2, NG4.2, R4.2
- net NOTE: now also R4.1; no longer NA4#.2, NA4.2, NB4.2, NC4#.2, NC4.2, ND4#.2, ND4.2, NE4.2, NF4#.2, NF4.2, NG4#.2, NG4.2
Routing:
- net KEYBOARD: track 0.00 -> 65.4 mm
- net NOTE: track 61.3 -> 5.21 mm
- net N$21: track 0.00 -> 8.00 mm
- net GND: track 125.7 -> 126.4 mm

Commit message: pots
Parts:
- removed R8: (no value), resistor:RTRIM5X
- added R5: (no value), pot:CA6V
- R1: device resistor:RTRIM5X -> pot:CA6V
- moved R1 31.5 mm to (52.0, 49.6), turned to 180 degrees
- moved SV2 2.43 mm to (9.95, 50.7)
Connections:
- net GND: now also R1.A, R5.A; no longer R1.1, R8.1
- net N$2: now also R1.E; no longer R8.3
- net N$5: now also R5.S; no longer R1.2
- net TONE: now also R5.E; no longer R1.3
- net VIBRATO: now also R1.S; no longer R8.2
Routing:
- net OUTPUT: track 7.62 -> 11.1 mm
- net NOTE: track 5.21 -> 8.50 mm
- net GND: track 126.4 -> 128.0 mm
- net N$5: track 5.93 -> 7.30 mm
- net N$2: track 10.8 -> 9.45 mm
- net VIBRATO: track 21.2 -> 20.2 mm
- net STYLUS: track 33.9 -> 34.5 mm
- net VCC: track 84.2 -> 84.8 mm

Commit message: bottom
Parts:
- R1, R5: device pot:CA6V -> pot:CA9V
- moved R1 8.10 mm to (45.2, 54.0), turned to 90 degrees
- moved IC2 4.00 mm to (7.08, 59.1)
- moved SV2 4.00 mm to (5.95, 50.7)
- moved R5 2.68 mm to (18.8, 53.6)
- moved NG4 2.53 mm to (42.5, 43.7), flipped to the bottom
- moved NG4# 2.53 mm to (47.6, 43.7), flipped to the bottom
- moved NC4 2.53 mm to (6.98, 43.7), flipped to the bottom
- moved ND4 2.53 mm to (17.1, 43.7), flipped to the bottom
- moved ND4# 2.53 mm to (22.2, 43.7), flipped to the bottom
- moved NE4 2.53 mm to (27.3, 43.7), flipped to the bottom
- moved NC4# 2.53 mm to (12.1, 43.7), flipped to the bottom
- moved NA4 2.53 mm to (52.7, 43.7), flipped to the bottom
- moved NA4# 2.53 mm to (57.8, 43.7), flipped to the bottom
- moved NB4 2.53 mm to (62.9, 43.7), flipped to the bottom
- moved NF4 2.53 mm to (32.4, 43.7), flipped to the bottom
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Routing:
- net VCC: track 84.8 -> 125.4 mm
- net STYLUS: track 34.5 -> 52.8 mm
- net VIBRATO: track 20.2 -> 5.68 mm
- net N$21: track 8.00 -> 0.00 mm
- net N$2: track 9.45 -> 4.09 mm
- net GND: track 128.0 -> 124.6 mm
- net N$7: track 0.00 -> 2.80 mm
- net OUTPUT: track 11.1 -> 8.29 mm
- net N$13: track 2.54 -> 0.00 mm
- net KEYBOARD: track 65.4 -> 62.8 mm
- net N$1: track 5.61 -> 4.63 mm
- net N$5: track 7.30 -> 7.99 mm
- net N$14: track 2.54 -> 3.20 mm
- net N$12: track 2.54 -> 3.20 mm
- net N$11: track 2.54 -> 3.20 mm
- added copper zone on layer 16, net N$10
- added copper zone on layer 16, net N$11
- added copper zone on layer 16, net N$12
- added copper zone on layer 16, net N$14
- added copper zone on layer 16, net N$15
- added copper zone on layer 16, net N$16
- added copper zone on layer 16, net N$17
- added copper zone on layer 16, net N$18
- added copper zone on layer 16, net N$19
- added copper zone on layer 16, net N$20
- added copper zone on layer 16, net N$7
- added copper zone on layer 16, net N$9
- removed copper zone on layer 1, net N$4
- removed copper zone on layer 1, net N$6
- removed copper zone on layer 1, net N$7
- removed copper zone on layer 1, net N$8
Other:
- board text added: "V"

Commit message: images
Other:
- board size 102.5 x 80 mm -> 75.3 x 41.2 mm

Commit message: done
Parts:
- R4: device rcl:0204/5 -> rcl:0204/7
- moved NC4 2.00 mm to (4.98, 43.7)
- moved NC4# 2.00 mm to (10.1, 43.7)
- moved ND4 1.60 mm to (15.5, 43.7)
- moved ND4# 1.60 mm to (20.6, 43.7)
- moved NB4 1.60 mm to (64.5, 43.7)
- moved NE4 1.20 mm to (26.1, 43.7)
- moved NA4# 1.20 mm to (59.0, 43.7)
- moved NF4 0.80 mm to (31.6, 43.7)
- moved NA4 0.80 mm to (53.5, 43.7)
- moved R4 0.57 mm to (38.0, 54.2)
- moved NG4# 0.40 mm to (48.0, 43.7)
- moved NF4# 0.40 mm to (37.1, 43.7)
Routing:
- net NG4#: track 0.00 -> 4.00 mm
- net NF4: track 0.00 -> 4.00 mm
- net NE4: track 0.00 -> 4.00 mm
- net ND4#: track 0.00 -> 4.00 mm
- net NA4: track 0.00 -> 4.00 mm
- net N$4: track 0.00 -> 3.86 mm
- net NG4: track 0.00 -> 3.60 mm
- net NF4#: track 0.00 -> 3.60 mm
- net ND4: track 0.00 -> 3.60 mm
- net NB4: track 0.00 -> 3.60 mm
- net NA4#: track 0.00 -> 3.60 mm
- net NC4#: track 0.00 -> 3.20 mm
- net NC4: track 0.00 -> 3.20 mm
- net N$14: track 3.20 -> 0.00 mm
- net N$12: track 3.20 -> 0.00 mm
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- added copper zone on layer 16, net NA4#
- added copper zone on layer 16, net NA4
- added copper zone on layer 16, net NB4
- added copper zone on layer 16, net NC4#
- added copper zone on layer 16, net NC4
- added copper zone on layer 16, net ND4#
- added copper zone on layer 16, net ND4
- added copper zone on layer 16, net NE4
- added copper zone on layer 16, net NF4#
- added copper zone on layer 16, net NF4
- added copper zone on layer 16, net NG4#
- added copper zone on layer 16, net NG4
- removed copper zone on layer 16, net N$10
- removed copper zone on layer 16, net N$11
- removed copper zone on layer 16, net N$12
- removed copper zone on layer 16, net N$14
- removed copper zone on layer 16, net N$15
- removed copper zone on layer 16, net N$16
- removed copper zone on layer 16, net N$17
- removed copper zone on layer 16, net N$18
- removed copper zone on layer 16, net N$19
- removed copper zone on layer 16, net N$20
- removed copper zone on layer 16, net N$7
- removed copper zone on layer 16, net N$9
Other:
- board text removed: "V"
