File: PCB/stylophone.sch (EAGLE design)
At the start: 25 parts, among them IC2 LM358N

Commit message: almost finished
Parts:
- removed R4: 100k, resistor:R-EU_M1206
- removed R5: 50k, resistor:R-EU_M1206
- removed R6: 1k, resistor:R-EU_M1206
- removed SV1: (no value), con-lstb:MA04-1
- added R1, R8: (no value), resistor:R-TRIMM5X
- added SV2: (no value), con-lstb:MA05-1
- R7: device resistor:R-EU_0204/7 -> resistor:R-EU_M1206
Connections:
- net GND: now also R1.E, R8.E, SV2.2, SV2.5; no longer R4.2, SV1.2, SV1.4
- net N$2: now also R8.A; no longer R6.2
- net N$5: now also R1.S; no longer R4.1, R5.2
- net OUTPUT: now also SV2.4; no longer SV1.3
- net STYLUS: now also SV2.3
- net TONE: now also R1.A; no longer R5.1
- net VCC: now also SV2.1; no longer SV1.1
- net VIBRATO: now also R8.S; no longer R6.1

Commit message: almost done
Parts:
- added R4: (no value), rcl:R-EU_0204/5
Connections:
- new net KEYBOARD: NA4#.2, NA4.2, NB4.2, NC4#.2, NC4.2, ND4#.2, ND4.2, NE4.2, NF4#.2, NF4.2, NG4#.2, NG4.2, R4.2
- net NOTE: now also R4.1; no longer NA4#.2, NA4.2, NB4.2, NC4#.2, NC4.2, ND4#.2, ND4.2, NE4.2, NF4#.2, NF4.2, NG4#.2, NG4.2
Changed lines of the file:
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@@
 <part name="R8" library="resistor" deviceset="R-TRIMM" device="5X"/>
 <part name="SV2" library="con-lstb" deviceset="MA05-1" device=""/>
+<part name="R4" library="rcl" deviceset="R-EU_" device="0204/5"/>
 </parts>
 <sheets>
@@
 <instance part="R8" gate="G$1" x="142.24" y="127"/>
 <instance part="SV2" gate="G$1" x="226.06" y="127" rot="R180"/>
+<instance part="R4" gate="G$1" x="25.4" y="86.36"/>
 </instances>
 <busses>
@@
 </segment>
 <segment>
+<pinref part="R4" gate="G$1" pin="1"/>
+<wire x1="20.32" y1="86.36" x2="12.7" y2="86.36" width="0.1524" layer="91"/>
+<label x="12.7" y="86.36" size="1.778" layer="95"/>
+</segment>
+</net>
+<net name="N$1" class="0">
+<segment>
+<pinref part="VIBRATO" gate="G$1" pin="CON"/>
+<wire x1="134.62" y1="121.92" x2="137.16" y2="121.92" width="0.1524" layer="91"/>
+<pinref part="C4" gate="G$1" pin="1"/>
+<wire x1="137.16" y1="121.92" x2="139.7" y2="119.38" width="0.1524" layer="91"/>
+</segment>
+</net>
+<net name="N$3" class="0">
+<segment>
+<pinref part="R7" gate="G$1" pin="1"/>
+<pinref part="R3" gate="G$1" pin="2"/>
+<wire x1="111.76" y1="144.78" x2="119.38" y2="144.78" width="0.1524" layer="91"/>
+<pinref part="VIBRATO" gate="G$1" pin="DIS"/>
+<wire x1="114.3" y1="127" x2="111.76" y2="127" width="0.1524" layer="91"/>
+<wire x1="111.76" y1="127" x2="111.76" y2="144.78" width="0.1524" layer="91"/>
+<junction x="111.76" y="144.78"/>
+</segment>
+</net>
+<net name="NOTSTYLUS" class="0">
+<segment>
+<pinref part="VIBRATO" gate="G$1" pin="TRI"/>
+<wire x1="114.3" y1="119.38" x2="109.22" y2="119.38" width="0.1524" layer="91"/>
+<wire x1="109.22" y1="119.38" x2="109.22" y2="134.62" width="0.1524" layer="91"/>
+<pinref part="VIBRATO" gate="G$1" pin="TRE"/>
+<wire x1="109.22" y1="134.62" x2="114.3" y2="134.62" width="0.1524" layer="91"/>
+<pinref part="C3" gate="G$1" pin="1"/>
+<wire x1="109.22" y1="134.62" x2="101.6" y2="134.62" width="0.1524" layer="91"/>
+<junction x="109.22" y="134.62"/>
+<pinref part="R7" gate="G$1" pin="2"/>
+<wire x1="101.6" y1="134.62" x2="99.06" y2="134.62" width="0.1524" layer="91"/>
+<wire x1="101.6" y1="144.78" x2="101.6" y2="134.62" width="0.1524" layer="91"/>
+<junction x="101.6" y="134.62"/>
+</segment>
+</net>
+<net name="N$2" class="0">
+<segment>
+<pinref part="VIBRATO" gate="G$1" pin="OUT"/>
+<wire x1="134.62" y1="127" x2="139.7" y2="132.08" width="0.1524" layer="91"/>
+<pinref part="R8" gate="G$1" pin="A"/>
+<wire x1="139.7" y1="132.08" x2="142.24" y2="132.08" width="0.1524" layer="91"/>
+</segment>
+</net>
+<net name="N$5" class="0">
+<segment>
+<pinref part="R1" gate="G$1" pin="S"/>
+<pinref part="IC2" gate="A" pin="+IN"/>
+<wire x1="182.88" y1="127" x2="185.42" y2="127" width="0.1524" layer="91"/>
+</segment>
+</net>
+<net name="KEYBOARD" class="0">
+<segment>
 <pinref part="NB4" gate="G$1" pin="2"/>
 <wire x1="157.48" y1="83.82" x2="154.94" y2="86.36" width="0.1524" layer="91"/>
-<label x="20.32" y="86.36" size="1.778" layer="95"/>
 <pinref part="NA4#" gate="G$1" pin="2"/>
 <wire x1="144.78" y1="83.82" x2="144.78" y2="86.36" width="0.1524" layer="91"/>
@@
 <wire x1="43.18" y1="86.36" x2="30.48" y2="86.36" width="0.1524" layer="91"/>
 <junction x="43.18" y="86.36"/>
-<wire x1="30.48" y1="86.36" x2="20.32" y2="86.36" width="0.1524" layer="91"/>
+<pinref part="R4" gate="G$1" pin="2"/>
 <junction x="30.48" y="86.36"/>
 </segment>
 </net>
-<net name="N$1" class="0">
-<segment>
-<pinref part="VIBRATO" gate="G$1" pin="CON"/>
-<wire x1="134.62" y1="121.92" x2="137.16" y2="121.92" width="0.1524" layer="91"/>
-<pinref part="C4" gate="G$1" pin="1"/>
-<wire x1="137.16" y1="121.92" x2="139.7" y2="119.38" width="0.1524" layer="91"/>
-</segment>
-</net>
-<net name="N$3" class="0">
-<segment>
-<pinref part="R7" gate="G$1" pin="1"/>
-<pinref part="R3" gate="G$1" pin="2"/>
-<wire x1="111.76" y1="144.78" x2="119.38" y2="144.78" width="0.1524" layer="91"/>
-<pinref part="VIBRATO" gate="G$1" pin="DIS"/>
-<wire x1="114.3" y1="127" x2="111.76" y2="127" width="0.1524" layer="91"/>
-<wire x1="111.76" y1="127" x2="111.76" y2="144.78" width="0.1524" layer="91"/>
-<junction x="111.76" y="144.78"/>
-</segment>
-</net>
-<net name="NOTSTYLUS" class="0">
-<segment>
-<pinref part="VIBRATO" gate="G$1" pin="TRI"/>
-<wire x1="114.3" y1="119.38" x2="109.22" y2="119.38" width="0.1524" layer="91"/>
-<wire x1="109.22" y1="119.38" x2="109.22" y2="134.62" width="0.1524" layer="91"/>
-<pinref part="VIBRATO" gate="G$1" pin="TRE"/>
-<wire x1="109.22" y1="134.62" x2="114.3" y2="134.62" width="0.1524" layer="91"/>
-<pinref part="C3" gate="G$1" pin="1"/>
-<wire x1="109.22" y1="134.62" x2="101.6" y2="134.62" width="0.1524" layer="91"/>
-<junction x="109.22" y="134.62"/>
-<pinref part="R7" gate="G$1" pin="2"/>
-<wire x1="101.6" y1="134.62" x2="99.06" y2="134.62" width="0.1524" layer="91"/>
-<wire x1="101.6" y1="144.78" x2="101.6" y2="134.62" width="0.1524" layer="91"/>
-<junction x="101.6" y="134.62"/>
-</segment>
-</net>
-<net name="N$2" class="0">
-<segment>
-<pinref part="VIBRATO" gate="G$1" pin="OUT"/>
-<wire x1="134.62" y1="127" x2="139.7" y2="132.08" width="0.1524" layer="91"/>
-<pinref part="R8" gate="G$1" pin="A"/>
-<wire x1="139.7" y1="132.08" x2="142.24" y2="132.08" width="0.1524" layer="91"/>
-</segment>
-</net>
-<net name="N$5" class="0">
-<segment>
-<pinref part="R1" gate="G$1" pin="S"/>
-<pinref part="IC2" gate="A" pin="+IN"/>
-<wire x1="182.88" y1="127" x2="185.42" y2="127" width="0.1524" layer="91"/>
-</segment>
-</net>

Commit message: pots
Parts:
- removed R8: (no value), resistor:R-TRIMM5X
- added R5: (no value), pot:TRIM_EU-CA6V
- R1: device resistor:R-TRIMM5X -> pot:TRIM_EU-CA6V
Connections:
- net GND: now also R1.A, R5.A; no longer R1.E, R8.E
- net N$2: now also R1.E; no longer R8.A
- net N$5: now also R5.S; no longer R1.S
- net TONE: now also R5.E; no longer R1.A
- net VIBRATO: now also R1.S; no longer R8.S
Changed lines of the file:
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@@
 <part name="NA4#" library="resistor" deviceset="R-EU_" device="M1206"/>
 <part name="NB4" library="resistor" deviceset="R-EU_" device="M1206"/>
-<part name="R1" library="resistor" deviceset="R-TRIMM" device="5X"/>
-<part name="R8" library="resistor" deviceset="R-TRIMM" device="5X"/>
 <part name="SV2" library="con-lstb" deviceset="MA05-1" device=""/>
 <part name="R4" library="rcl" deviceset="R-EU_" device="0204/5"/>
+<part name="R5" library="pot" deviceset="TRIM_EU-" device="CA6V"/>
+<part name="R1" library="pot" deviceset="TRIM_EU-" device="CA6V"/>
 </parts>
 <sheets>
@@
 <instance part="NA4#" gate="G$1" x="144.78" y="78.74" rot="R90"/>
 <instance part="NB4" gate="G$1" x="157.48" y="78.74" rot="R90"/>
-<instance part="R1" gate="G$1" x="177.8" y="127"/>
-<instance part="R8" gate="G$1" x="142.24" y="127"/>
 <instance part="SV2" gate="G$1" x="226.06" y="127" rot="R180"/>
 <instance part="R4" gate="G$1" x="25.4" y="86.36"/>
+<instance part="R5" gate="1" x="177.8" y="127"/>
+<instance part="R1" gate="1" x="142.24" y="127"/>
 </instances>
 <busses>
@@
 <segment>
 <wire x1="213.36" y1="121.92" x2="205.74" y2="114.3" width="0.1524" layer="91"/>
-<pinref part="R1" gate="G$1" pin="E"/>
 <wire x1="177.8" y1="121.92" x2="177.8" y2="116.84" width="0.1524" layer="91"/>
 <wire x1="177.8" y1="116.84" x2="180.34" y2="114.3" width="0.1524" layer="91"/>
 <wire x1="180.34" y1="114.3" x2="205.74" y2="114.3" width="0.1524" layer="91"/>
+<pinref part="R5" gate="1" pin="A"/>
 </segment>
 <segment>
@@
 <wire x1="134.62" y1="111.76" x2="139.7" y2="111.76" width="0.1524" layer="91"/>
 <label x="134.62" y="109.22" size="1.778" layer="95"/>
-<pinref part="R8" gate="G$1" pin="E"/>
 <wire x1="142.24" y1="121.92" x2="147.32" y2="116.84" width="0.1524" layer="91"/>
 <wire x1="147.32" y1="116.84" x2="147.32" y2="111.76" width="0.1524" layer="91"/>
 <wire x1="147.32" y1="111.76" x2="139.7" y2="111.76" width="0.1524" layer="91"/>
 <junction x="139.7" y="111.76"/>
+<pinref part="R1" gate="1" pin="A"/>
 </segment>
 <segment>
@@
 </segment>
 <segment>
-<pinref part="R1" gate="G$1" pin="A"/>
 <wire x1="177.8" y1="132.08" x2="180.34" y2="134.62" width="0.1524" layer="91"/>
 <wire x1="180.34" y1="134.62" x2="187.96" y2="134.62" width="0.1524" layer="91"/>
 <label x="180.34" y="134.62" size="1.778" layer="95"/>
+<pinref part="R5" gate="1" pin="E"/>
 </segment>
 </net>
@@
 </segment>
 <segment>
-<pinref part="R8" gate="G$1" pin="S"/>
 <wire x1="147.32" y1="127" x2="154.94" y2="127" width="0.1524" layer="91"/>
 <label x="147.32" y="127" size="1.778" layer="95"/>
+<pinref part="R1" gate="1" pin="S"/>
 </segment>
 </net>
@@
 <pinref part="VIBRATO" gate="G$1" pin="OUT"/>
 <wire x1="134.62" y1="127" x2="139.7" y2="132.08" width="0.1524" layer="91"/>
-<pinref part="R8" gate="G$1" pin="A"/>
 <wire x1="139.7" y1="132.08" x2="142.24" y2="132.08" width="0.1524" layer="91"/>
+<pinref part="R1" gate="1" pin="E"/>
 </segment>
 </net>
 <net name="N$5" class="0">
 <segment>
-<pinref part="R1" gate="G$1" pin="S"/>
 <pinref part="IC2" gate="A" pin="+IN"/>
 <wire x1="182.88" y1="127" x2="185.42" y2="127" width="0.1524" layer="91"/>
-</segment>
-</net>
+<pinref part="R5" gate="1" pin="S"/>
+</segment>
+</net>

Commit message: bottom
Parts:
- R1, R5: device pot:TRIM_EU-CA6V -> pot:TRIM_EU-CA9V
Changed lines of the file:
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@@
 <part name="SV2" library="con-lstb" deviceset="MA05-1" device=""/>
 <part name="R4" library="rcl" deviceset="R-EU_" device="0204/5"/>
-<part name="R5" library="pot" deviceset="TRIM_EU-" device="CA6V"/>
-<part name="R1" library="pot" deviceset="TRIM_EU-" device="CA6V"/>
+<part name="R5" library="pot" deviceset="TRIM_EU-" device="CA9V"/>
+<part name="R1" library="pot" deviceset="TRIM_EU-" device="CA9V"/>
 </parts>
 <sheets>

Commit message: done
Parts:
- R4: device rcl:R-EU_0204/5 -> rcl:R-EU_0204/7
Changed lines of the file:
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@@
 <grid distance="0.1" unitdist="inch" unit="inch" style="lines" multiple="1" display="no" altdistance="0.01" altunitdist="inch" altunit="inch"/>
 <layers>
-<layer number="1" name="Top" color="4" fill="1" visible="no" active="no"/>
-<layer number="16" name="Bottom" color="1" fill="1" visible="no" active="no"/>
-<layer number="17" name="Pads" color="2" fill="1" visible="no" active="no"/>
-<layer number="18" name="Vias" color="2" fill="1" visible="no" active="no"/>
-<layer number="19" name="Unrouted" color="6" fill="1" visible="no" active="no"/>
-<layer number="20" name="Dimension" color="15" fill="1" visible="no" active="no"/>
-<layer number="21" name="tPlace" color="7" fill="1" visible="no" active="no"/>
-<layer number="22" name="bPlace" color="7" fill="1" visible="no" active="no"/>
-<layer number="23" name="tOrigins" color="15" fill="1" visible="no" active="no"/>
-<layer number="24" name="bOrigins" color="15" fill="1" visible="no" active="no"/>
-<layer number="25" name="tNames" color="7" fill="1" visible="no" active="no"/>
-<layer number="26" name="bNames" color="7" fill="1" visible="no" active="no"/>
-<layer number="27" name="tValues" color="7" fill="1" visible="no" active="no"/>
-<layer number="28" name="bValues" color="7" fill="1" visible="no" active="no"/>
+<layer number="1" name="Top" color="4" fill="1" visible="yes" active="no"/>
+<layer number="16" name="Bottom" color="1" fill="1" visible="yes" active="no"/>
+<layer number="17" name="Pads" color="2" fill="1" visible="yes" active="no"/>
+<layer number="18" name="Vias" color="2" fill="1" visible="yes" active="no"/>
+<layer number="19" name="Unrouted" color="6" fill="1" visible="yes" active="no"/>
+<layer number="20" name="Dimension" color="15" fill="1" visible="yes" active="no"/>
+<layer number="21" name="tPlace" color="15" fill="1" visible="yes" active="no"/>
+<layer number="22" name="bPlace" color="15" fill="1" visible="yes" active="no"/>
+<layer number="23" name="tOrigins" color="15" fill="1" visible="yes" active="no"/>
+<layer number="24" name="bOrigins" color="15" fill="1" visible="yes" active="no"/>
+<layer number="25" name="tNames" color="15" fill="1" visible="yes" active="no"/>
+<layer number="26" name="bNames" color="15" fill="1" visible="yes" active="no"/>
+<layer number="27" name="tValues" color="15" fill="1" visible="yes" active="no"/>
+<layer number="28" name="bValues" color="15" fill="1" visible="yes" active="no"/>
 <layer number="29" name="tStop" color="7" fill="3" visible="no" active="no"/>
 <layer number="30" name="bStop" color="7" fill="6" visible="no" active="no"/>
@@
 <layer number="35" name="tGlue" color="7" fill="4" visible="no" active="no"/>
 <layer number="36" name="bGlue" color="7" fill="5" visible="no" active="no"/>
-<layer number="37" name="tTest" color="7" fill="1" visible="no" active="no"/>
-<layer number="38" name="bTest" color="7" fill="1" visible="no" active="no"/>
+<layer number="37" name="tTest" color="7" fill="1" visible="yes" active="no"/>
+<layer number="38" name="bTest" color="7" fill="1" visible="yes" active="no"/>
 <layer number="39" name="tKeepout" color="4" fill="11" visible="no" active="no"/>
 <layer number="40" name="bKeepout" color="1" fill="11" visible="no" active="no"/>
@@
 <layer number="44" name="Drills" color="7" fill="1" visible="no" active="no"/>
 <layer number="45" name="Holes" color="7" fill="1" visible="no" active="no"/>
-<layer number="46" name="Milling" color="3" fill="1" visible="no" active="no"/>
-<layer number="47" name="Measures" color="7" fill="1" visible="no" active="no"/>
-<layer number="48" name="Document" color="7" fill="1" visible="no" active="no"/>
-<layer number="49" name="Reference" color="7" fill="1" visible="no" active="no"/>
-<layer number="51" name="tDocu" color="7" fill="1" visible="no" active="no"/>
-<layer number="52" name="bDocu" color="7" fill="1" visible="no" active="no"/>
+<layer number="46" name="Milling" color="3" fill="1" visible="yes" active="no"/>
+<layer number="47" name="Measures" color="7" fill="1" visible="yes" active="no"/>
+<layer number="48" name="Document" color="7" fill="1" visible="yes" active="no"/>
+<layer number="49" name="Reference" color="7" fill="1" visible="yes" active="no"/>
+<layer number="51" name="tDocu" color="7" fill="1" visible="yes" active="no"/>
+<layer number="52" name="bDocu" color="7" fill="1" visible="yes" active="no"/>
 <layer number="91" name="Nets" color="2" fill="1" visible="yes" active="yes"/>
 <layer number="92" name="Busses" color="1" fill="1" visible="yes" active="yes"/>
@@
 <part name="NB4" library="resistor" deviceset="R-EU_" device="M1206"/>
 <part name="SV2" library="con-lstb" deviceset="MA05-1" device=""/>
-<part name="R4" library="rcl" deviceset="R-EU_" device="0204/5"/>
+<part name="R4" library="rcl" deviceset="R-EU_" device="0204/7"/>
 <part name="R5" library="pot" deviceset="TRIM_EU-" device="CA9V"/>
 <part name="R1" library="pot" deviceset="TRIM_EU-" device="CA9V"/>
