File: PCB/pomiary.sch (EAGLE design)
At the start: 17 parts, among them IC2 LM358N

Commit message: almost finished
Parts:
- removed R5: 50k, resistor:R-EU_M1206
- removed R6: 1k, resistor:R-EU_M1206
- added R1: (no value), resistor:R-TRIMM5X
- R4: value 100k -> (none); device resistor:R-EU_M1206 -> resistor:R-TRIMM5X
Connections:
- removed net N$2: R6.2, VIBRATO.OUT
- new net N$4: R4.A, VIBRATO.OUT
- net GND: now also R1.E, R4.E; no longer R4.2
- net N$5: now also R1.S; no longer R4.1, R5.2
- net TONE: now also R1.A; no longer R5.1
- net VIBRATO: now also R4.S; no longer R6.1
Changed lines of the file:
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@@
 <part name="TONE" library="st-microelectronics" deviceset="NE555" device=""/>
 <part name="IC2" library="linear" deviceset="LM358" device="N"/>
-<part name="R4" library="resistor" deviceset="R-EU_" device="M1206" value="100k"/>
-<part name="R5" library="resistor" deviceset="R-EU_" device="M1206" value="50k"/>
 <part name="R2" library="resistor" deviceset="R-EU_" device="M1206" value="1k"/>
 <part name="C2" library="capacitor-wima" deviceset="C" device="2.5/5" value="100n"/>
@@
 <part name="C3" library="capacitor-wima" deviceset="C" device="2.5/5" value="1u"/>
 <part name="C4" library="capacitor-wima" deviceset="C" device="2.5/5" value="10n"/>
-<part name="R6" library="resistor" deviceset="R-EU_" device="M1206" value="1k"/>
 <part name="R7" library="resistor" deviceset="R-EU_" device="0204/7" value="10k"/>
 <part name="U$3" library="Przyrzady pomiarowe" deviceset="OSCYLOSKOP_AC_AC" device=""/>
@@
 <part name="U$4" library="Przyrzady pomiarowe" deviceset="OSCYLOSKOP_AC_AC" device=""/>
 <part name="SUPPLY4" library="supply2" deviceset="GND" device=""/>
+<part name="R1" library="resistor" deviceset="R-TRIMM" device="5X"/>
+<part name="R4" library="resistor" deviceset="R-TRIMM" device="5X"/>
 </parts>
 <sheets>
@@
 <instance part="TONE" gate="G$1" x="-271.78" y="121.92"/>
 <instance part="IC2" gate="A" x="-147.32" y="114.3"/>
-<instance part="R4" gate="G$1" x="-165.1" y="116.84" rot="R180"/>
-<instance part="R5" gate="G$1" x="-157.48" y="124.46" rot="R270"/>
 <instance part="R2" gate="G$1" x="-271.78" y="139.7" rot="R180"/>
 <instance part="C2" gate="G$1" x="-302.26" y="127"/>
@@
 <instance part="C3" gate="G$1" x="-243.84" y="127"/>
 <instance part="C4" gate="G$1" x="-203.2" y="111.76"/>
-<instance part="R6" gate="G$1" x="-200.66" y="121.92" rot="R180"/>
 <instance part="R7" gate="G$1" x="-236.22" y="139.7" rot="R180"/>
 <instance part="U$3" gate="G$1" x="-149.86" y="144.78"/>
@@
 <instance part="U$4" gate="G$1" x="-274.32" y="165.1"/>
 <instance part="SUPPLY4" gate="GND" x="-259.08" y="147.32"/>
+<instance part="R1" gate="G$1" x="-162.56" y="116.84"/>
+<instance part="R4" gate="G$1" x="-200.66" y="121.92"/>
 </instances>
 <busses>
@@
 <segment>
 <pinref part="IC2" gate="A" pin="+IN"/>
-<pinref part="R4" gate="G$1" pin="1"/>
 <wire x1="-154.94" y1="116.84" x2="-157.48" y2="116.84" width="0.1524" layer="91"/>
-<pinref part="R5" gate="G$1" pin="2"/>
-<wire x1="-157.48" y1="116.84" x2="-160.02" y2="116.84" width="0.1524" layer="91"/>
-<wire x1="-157.48" y1="119.38" x2="-157.48" y2="116.84" width="0.1524" layer="91"/>
-<junction x="-157.48" y="116.84"/>
 <pinref part="U$3" gate="G$1" pin="CH1"/>
 <wire x1="-149.86" y1="132.08" x2="-149.86" y2="124.46" width="0.1524" layer="91"/>
 <wire x1="-149.86" y1="124.46" x2="-157.48" y2="116.84" width="0.1524" layer="91"/>
+<pinref part="R1" gate="G$1" pin="S"/>
+<junction x="-157.48" y="116.84"/>
 </segment>
 </net>
 <net name="GND" class="0">
-<segment>
-<pinref part="R4" gate="G$1" pin="2"/>
-<label x="-175.26" y="116.84" size="1.778" layer="95"/>
-<wire x1="-170.18" y1="116.84" x2="-175.26" y2="116.84" width="0.1524" layer="91"/>
-</segment>
 <segment>
 <pinref part="SUPPLY1" gate="GND" pin="GND"/>
@@
 <wire x1="-208.28" y1="106.68" x2="-203.2" y2="106.68" width="0.1524" layer="91"/>
 <label x="-208.28" y="104.14" size="1.778" layer="95"/>
+<wire x1="-195.58" y1="106.68" x2="-203.2" y2="106.68" width="0.1524" layer="91"/>
+<junction x="-203.2" y="106.68"/>
+<pinref part="R4" gate="G$1" pin="E"/>
+<wire x1="-200.66" y1="116.84" x2="-195.58" y2="111.76" width="0.1524" layer="91"/>
+<wire x1="-195.58" y1="111.76" x2="-195.58" y2="106.68" width="0.1524" layer="91"/>
 </segment>
 <segment>
@@
 <wire x1="-121.92" y1="111.76" x2="-129.54" y2="111.76" width="0.1524" layer="91"/>
 <label x="-129.54" y="111.76" size="1.778" layer="95"/>
+<pinref part="R1" gate="G$1" pin="E"/>
+<wire x1="-162.56" y1="111.76" x2="-162.56" y2="106.68" width="0.1524" layer="91"/>
+<wire x1="-162.56" y1="106.68" x2="-160.02" y2="104.14" width="0.1524" layer="91"/>
+<wire x1="-160.02" y1="104.14" x2="-137.16" y2="104.14" width="0.1524" layer="91"/>
+<wire x1="-137.16" y1="104.14" x2="-129.54" y2="111.76" width="0.1524" layer="91"/>
 </segment>
 <segment>
@@
 </net>
 <net name="TONE" class="0">
-<segment>
-<pinref part="R5" gate="G$1" pin="1"/>
-<wire x1="-157.48" y1="129.54" x2="-160.02" y2="132.08" width="0.1524" layer="91"/>
-<wire x1="-160.02" y1="132.08" x2="-162.56" y2="132.08" width="0.1524" layer="91"/>
-<label x="-165.1" y="132.08" size="1.778" layer="95"/>
-</segment>
 <segment>
 <pinref part="TONE" gate="G$1" pin="OUT"/>
@@
 <wire x1="-266.7" y1="144.78" x2="-266.7" y2="152.4" width="0.1524" layer="91"/>
 </segment>
+<segment>
+<pinref part="R1" gate="G$1" pin="A"/>
+<wire x1="-162.56" y1="121.92" x2="-160.02" y2="124.46" width="0.1524" layer="91"/>
+<wire x1="-160.02" y1="124.46" x2="-152.4" y2="124.46" width="0.1524" layer="91"/>
+<label x="-160.02" y="124.46" size="1.778" layer="95"/>
+</segment>
 </net>
 <net name="VIBRATO" class="0">
@@
 </segment>
 <segment>
-<pinref part="R6" gate="G$1" pin="1"/>
-<wire x1="-195.58" y1="121.92" x2="-185.42" y2="121.92" width="0.1524" layer="91"/>
-<junction x="-195.58" y="121.92"/>
-<label x="-195.58" y="121.92" size="1.778" layer="95"/>
+<pinref part="R4" gate="G$1" pin="S"/>
+<wire x1="-195.58" y1="121.92" x2="-195.58" y2="127" width="0.1524" layer="91"/>
 <pinref part="U$2" gate="G$1" pin="CH2"/>
 <wire x1="-208.28" y1="152.4" x2="-208.28" y2="142.24" width="0.1524" layer="91"/>
-<wire x1="-208.28" y1="142.24" x2="-200.66" y2="134.62" width="0.1524" layer="91"/>
-<wire x1="-200.66" y1="134.62" x2="-198.12" y2="134.62" width="0.1524" layer="91"/>
-<wire x1="-198.12" y1="134.62" x2="-195.58" y2="132.08" width="0.1524" layer="91"/>
-<wire x1="-195.58" y1="132.08" x2="-195.58" y2="121.92" width="0.1524" layer="91"/>
+<wire x1="-195.58" y1="127" x2="-208.28" y2="142.24" width="0.1524" layer="91"/>
+<wire x1="-195.58" y1="121.92" x2="-182.88" y2="121.92" width="0.1524" layer="91"/>
+<junction x="-195.58" y="121.92"/>
+<label x="-193.04" y="121.92" size="1.778" layer="95"/>
 </segment>
 </net>
@@
 <pinref part="C4" gate="G$1" pin="1"/>
 <wire x1="-205.74" y1="116.84" x2="-203.2" y2="114.3" width="0.1524" layer="91"/>
-</segment>
-</net>
-<net name="N$2" class="0">
-<segment>
-<pinref part="VIBRATO" gate="G$1" pin="OUT"/>
-<pinref part="R6" gate="G$1" pin="2"/>
-<wire x1="-208.28" y1="121.92" x2="-205.74" y2="121.92" width="0.1524" layer="91"/>
 </segment>
 </net>
@@
 </segment>
 </net>
+<net name="N$4" class="0">
+<segment>
+<pinref part="VIBRATO" gate="G$1" pin="OUT"/>
+<wire x1="-208.28" y1="121.92" x2="-203.2" y2="127" width="0.1524" layer="91"/>
+<pinref part="R4" gate="G$1" pin="A"/>
+<wire x1="-203.2" y1="127" x2="-200.66" y2="127" width="0.1524" layer="91"/>
+</segment>
+</net>

Commit message: images
Connections:
- net GND: now also TONE.GND
Changed lines of the file:
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@@
 <part name="R1" library="resistor" deviceset="R-TRIMM" device="5X"/>
 <part name="R4" library="resistor" deviceset="R-TRIMM" device="5X"/>
+<part name="FRAME1" library="frames" deviceset="A4L-LOC" device=""/>
 </parts>
 <sheets>
@@
 </plain>
 <instances>
-<instance part="TONE" gate="G$1" x="-271.78" y="121.92"/>
-<instance part="IC2" gate="A" x="-147.32" y="114.3"/>
-<instance part="R2" gate="G$1" x="-271.78" y="139.7" rot="R180"/>
-<instance part="C2" gate="G$1" x="-302.26" y="127"/>
-<instance part="SUPPLY1" gate="GND" x="-302.26" y="116.84"/>
-<instance part="VIBRATO" gate="G$1" x="-218.44" y="121.92"/>
-<instance part="R3" gate="G$1" x="-218.44" y="139.7" rot="R180"/>
-<instance part="C3" gate="G$1" x="-243.84" y="127"/>
-<instance part="C4" gate="G$1" x="-203.2" y="111.76"/>
-<instance part="R7" gate="G$1" x="-236.22" y="139.7" rot="R180"/>
-<instance part="U$3" gate="G$1" x="-149.86" y="144.78"/>
-<instance part="SV2" gate="1" x="-114.3" y="114.3" rot="R180"/>
-<instance part="U$1" gate="G$1" x="-109.22" y="147.32"/>
-<instance part="SUPPLY2" gate="GND" x="-119.38" y="127"/>
-<instance part="U$2" gate="G$1" x="-215.9" y="165.1"/>
-<instance part="SUPPLY3" gate="GND" x="-200.66" y="147.32"/>
-<instance part="U$4" gate="G$1" x="-274.32" y="165.1"/>
-<instance part="SUPPLY4" gate="GND" x="-259.08" y="147.32"/>
-<instance part="R1" gate="G$1" x="-162.56" y="116.84"/>
-<instance part="R4" gate="G$1" x="-200.66" y="121.92"/>
+<instance part="TONE" gate="G$1" x="-271.78" y="121.92" smashed="yes">
+<attribute name="NAME" x="-279.4" y="133.35" size="1.778" layer="95"/>
+<attribute name="VALUE" x="-279.4" y="109.22" size="1.778" layer="96"/>
+</instance>
+<instance part="IC2" gate="A" x="-147.32" y="114.3" smashed="yes">
+<attribute name="NAME" x="-144.78" y="117.475" size="1.778" layer="95"/>
+<attribute name="VALUE" x="-144.78" y="109.22" size="1.778" layer="96"/>
+</instance>
+<instance part="R2" gate="G$1" x="-271.78" y="139.7" smashed="yes" rot="R180">
+<attribute name="NAME" x="-267.97" y="138.2014" size="1.778" layer="95" rot="R180"/>
+<attribute name="VALUE" x="-267.97" y="143.002" size="1.778" layer="96" rot="R180"/>
+</instance>
+<instance part="C2" gate="G$1" x="-302.26" y="127" smashed="yes">
+<attribute name="NAME" x="-300.736" y="127.381" size="1.778" layer="95"/>
+<attribute name="VALUE" x="-300.736" y="122.301" size="1.778" layer="96"/>
+</instance>
+<instance part="SUPPLY1" gate="GND" x="-302.26" y="116.84" smashed="yes">
+<attribute name="VALUE" x="-304.165" y="113.665" size="1.778" layer="96"/>
+</instance>
+<instance part="VIBRATO" gate="G$1" x="-218.44" y="121.92" smashed="yes">
+<attribute name="NAME" x="-226.06" y="133.35" size="1.778" layer="95"/>
+<attribute name="VALUE" x="-226.06" y="109.22" size="1.778" layer="96"/>
+</instance>
+<instance part="R3" gate="G$1" x="-218.44" y="139.7" smashed="yes" rot="R180">
+<attribute name="NAME" x="-214.63" y="138.2014" size="1.778" layer="95" rot="R180"/>
+<attribute name="VALUE" x="-214.63" y="143.002" size="1.778" layer="96" rot="R180"/>
+</instance>
+<instance part="C3" gate="G$1" x="-243.84" y="127" smashed="yes">
+<attribute name="NAME" x="-242.316" y="127.381" size="1.778" layer="95"/>
+<attribute name="VALUE" x="-242.316" y="122.301" size="1.778" layer="96"/>
+</instance>
+<instance part="C4" gate="G$1" x="-203.2" y="111.76" smashed="yes">
+<attribute name="NAME" x="-201.676" y="112.141" size="1.778" layer="95"/>
+<attribute name="VALUE" x="-201.676" y="107.061" size="1.778" layer="96"/>
+</instance>
+<instance part="R7" gate="G$1" x="-236.22" y="139.7" smashed="yes" rot="R180">
+<attribute name="NAME" x="-232.41" y="138.2014" size="1.778" layer="95" rot="R180"/>
+<attribute name="VALUE" x="-232.41" y="143.002" size="1.778" layer="96" rot="R180"/>
+</instance>
+<instance part="U$3" gate="G$1" x="-149.86" y="144.78" smashed="yes"/>
+<instance part="SV2" gate="1" x="-114.3" y="114.3" smashed="yes" rot="R180">
+<attribute name="VALUE" x="-113.03" y="124.46" size="1.778" layer="96" rot="R180"/>
+<attribute name="NAME" x="-113.03" y="108.458" size="1.778" layer="95" rot="R180"/>
+</instance>
+<instance part="U$1" gate="G$1" x="-109.22" y="147.32" smashed="yes"/>
+<instance part="SUPPLY2" gate="GND" x="-119.38" y="127" smashed="yes">
+<attribute name="VALUE" x="-121.285" y="123.825" size="1.778" layer="96"/>
+</instance>
+<instance part="U$2" gate="G$1" x="-215.9" y="165.1" smashed="yes"/>
+<instance part="SUPPLY3" gate="GND" x="-200.66" y="147.32" smashed="yes">
+<attribute name="VALUE" x="-202.565" y="144.145" size="1.778" layer="96"/>
+</instance>
+<instance part="U$4" gate="G$1" x="-274.32" y="165.1" smashed="yes"/>
+<instance part="SUPPLY4" gate="GND" x="-259.08" y="147.32" smashed="yes">
+<attribute name="VALUE" x="-260.985" y="144.145" size="1.778" layer="96"/>
+</instance>
+<instance part="R1" gate="G$1" x="-162.56" y="116.84" smashed="yes">
+<attribute name="NAME" x="-166.37" y="115.951" size="1.778" layer="95" rot="R180"/>
+<attribute name="VALUE" x="-166.37" y="113.03" size="1.778" layer="96" rot="R90"/>
+</instance>
+<instance part="R4" gate="G$1" x="-200.66" y="121.92" smashed="yes">
+<attribute name="NAME" x="-204.47" y="121.031" size="1.778" layer="95" rot="R180"/>
+<attribute name="VALUE" x="-204.47" y="118.11" size="1.778" layer="96" rot="R90"/>
+</instance>
+<instance part="FRAME1" gate="G$1" x="-330.2" y="53.34"/>
 </instances>
 <busses>
@@
 <wire x1="-259.08" y1="149.86" x2="-259.08" y2="152.4" width="0.1524" layer="91"/>
 </segment>
-</net>
+<segment>
+<pinref part="TONE" gate="G$1" pin="GND"/>
+<wire x1="-261.62" y1="114.3" x2="-259.08" y2="111.76" width="0.1524" layer="91"/>
+<wire x1="-259.08" y1="111.76" x2="-259.08" y2="109.22" width="0.1524" layer="91"/>
+<label x="-259.08" y="109.22" size="1.778" layer="95"/>
+</segment>
+</net>

Commit message: frfr
Connections:
- removed net N$5: IC2A.+IN, R1.S, U$3.CH1
- new net N$2: IC2A.+IN, R1.S
- net NOTSTYLUS: no longer U$2.CH1
- net OUTPUT: no longer U$3.CH2
- net STYLUS: no longer U$4.CH1
- net TONE: no longer U$4.CH2
- net VIBRATO: no longer U$2.CH2
Other:
- note added: "Pomiar przebiegu ładowania kondensatora Tone pomiar przebiegu wyjścia Tone"
- note added: "Pomiar przebiegu ładowania kondensatora Vibrato pomiar wpływu potencjometru Vibrato na wyjście Vibrato oraz Tone"
- note added: "Pomiar wpływu potencjometru Volume na wyjście"
Changed lines of the file:
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@@
 <layer number="93" name="Pins" color="2" fill="1" visible="no" active="yes"/>
 <layer number="94" name="Symbols" color="4" fill="1" visible="yes" active="yes"/>
-<layer number="95" name="Names" color="7" fill="1" visible="yes" active="yes"/>
+<layer number="95" name="Names" color="15" fill="1" visible="yes" active="yes"/>
 <layer number="96" name="Values" color="7" fill="1" visible="yes" active="yes"/>
 <layer number="97" name="Info" color="7" fill="1" visible="yes" active="yes"/>
@@
 <sheet>
 <plain>
+<text x="-289.56" y="180.34" size="1.778" layer="95">Pomiar przebiegu ładowania kondensatora Tone
+pomiar przebiegu wyjścia Tone</text>
+<text x="-231.14" y="180.34" size="1.778" layer="95">Pomiar przebiegu ładowania kondensatora Vibrato
+pomiar wpływu potencjometru Vibrato na wyjście Vibrato oraz Tone</text>
+<text x="-157.48" y="180.34" size="1.778" layer="95">Pomiar wpływu potencjometru Volume na wyjście</text>
 </plain>
 <instances>
@@
 </instances>
 <busses>
+<bus name="B$1">
+<segment>
+<wire x1="-274.32" y1="152.4" x2="-294.64" y2="152.4" width="0.762" layer="92"/>
+<wire x1="-294.64" y1="152.4" x2="-302.26" y2="144.78" width="0.762" layer="92"/>
+<wire x1="-302.26" y1="144.78" x2="-302.26" y2="129.54" width="0.762" layer="92"/>
+</segment>
+</bus>
+<bus name="B$2">
+<segment>
+<wire x1="-266.7" y1="152.4" x2="-266.7" y2="144.78" width="0.762" layer="92"/>
+<wire x1="-266.7" y1="144.78" x2="-259.08" y2="137.16" width="0.762" layer="92"/>
+<wire x1="-259.08" y1="137.16" x2="-259.08" y2="121.92" width="0.762" layer="92"/>
+</segment>
+</bus>
+<bus name="B$3">
+<segment>
+<wire x1="-243.84" y1="129.54" x2="-243.84" y2="147.32" width="0.762" layer="92"/>
+<wire x1="-243.84" y1="147.32" x2="-238.76" y2="152.4" width="0.762" layer="92"/>
+<wire x1="-238.76" y1="152.4" x2="-215.9" y2="152.4" width="0.762" layer="92"/>
+</segment>
+</bus>
+<bus name="B$4">
+<segment>
+<wire x1="-208.28" y1="152.4" x2="-208.28" y2="144.78" width="0.762" layer="92"/>
+<wire x1="-208.28" y1="144.78" x2="-195.58" y2="132.08" width="0.762" layer="92"/>
+<wire x1="-195.58" y1="132.08" x2="-195.58" y2="121.92" width="0.762" layer="92"/>
+</segment>
+</bus>
+<bus name="B$5">
+<segment>
+<wire x1="-154.94" y1="116.84" x2="-154.94" y2="119.38" width="0.762" layer="92"/>
+<wire x1="-154.94" y1="119.38" x2="-149.86" y2="124.46" width="0.762" layer="92"/>
+<wire x1="-149.86" y1="124.46" x2="-149.86" y2="132.08" width="0.762" layer="92"/>
+</segment>
+</bus>
+<bus name="B$6">
+<segment>
+<wire x1="-142.24" y1="132.08" x2="-142.24" y2="127" width="0.762" layer="92"/>
+<wire x1="-142.24" y1="127" x2="-132.08" y2="116.84" width="0.762" layer="92"/>
+<wire x1="-132.08" y1="116.84" x2="-124.46" y2="116.84" width="0.762" layer="92"/>
+<wire x1="-124.46" y1="116.84" x2="-121.92" y2="114.3" width="0.762" layer="92"/>
+</segment>
+</bus>
 </busses>
 <nets>
@@
 <wire x1="-134.62" y1="114.3" x2="-121.92" y2="114.3" width="0.1524" layer="91"/>
 <junction x="-134.62" y="114.3"/>
-<pinref part="U$3" gate="G$1" pin="CH2"/>
-<wire x1="-142.24" y1="132.08" x2="-142.24" y2="124.46" width="0.1524" layer="91"/>
-<wire x1="-142.24" y1="124.46" x2="-134.62" y2="116.84" width="0.1524" layer="91"/>
-<wire x1="-134.62" y1="116.84" x2="-124.46" y2="116.84" width="0.1524" layer="91"/>
-<wire x1="-124.46" y1="116.84" x2="-121.92" y2="114.3" width="0.1524" layer="91"/>
-<junction x="-121.92" y="114.3"/>
 <label x="-134.62" y="114.3" size="1.778" layer="95"/>
-</segment>
-</net>
-<net name="N$5" class="0">
-<segment>
-<pinref part="IC2" gate="A" pin="+IN"/>
-<wire x1="-154.94" y1="116.84" x2="-157.48" y2="116.84" width="0.1524" layer="91"/>
-<pinref part="U$3" gate="G$1" pin="CH1"/>
-<wire x1="-149.86" y1="132.08" x2="-149.86" y2="124.46" width="0.1524" layer="91"/>
-<wire x1="-149.86" y1="124.46" x2="-157.48" y2="116.84" width="0.1524" layer="91"/>
-<pinref part="R1" gate="G$1" pin="S"/>
-<junction x="-157.48" y="116.84"/>
 </segment>
 </net>
@@
 <pinref part="TONE" gate="G$1" pin="OUT"/>
 <label x="-259.08" y="121.92" size="1.778" layer="95"/>
-<wire x1="-261.62" y1="121.92" x2="-259.08" y2="121.92" width="0.1524" layer="91"/>
-<wire x1="-259.08" y1="121.92" x2="-251.46" y2="121.92" width="0.1524" layer="91"/>
-<wire x1="-259.08" y1="121.92" x2="-259.08" y2="137.16" width="0.1524" layer="91"/>
-<junction x="-259.08" y="121.92"/>
-<wire x1="-259.08" y1="137.16" x2="-266.7" y2="144.78" width="0.1524" layer="91"/>
-<pinref part="U$4" gate="G$1" pin="CH2"/>
-<wire x1="-266.7" y1="144.78" x2="-266.7" y2="152.4" width="0.1524" layer="91"/>
+<wire x1="-261.62" y1="121.92" x2="-251.46" y2="121.92" width="0.1524" layer="91"/>
 </segment>
 <segment>
@@
 <segment>
 <pinref part="R4" gate="G$1" pin="S"/>
-<wire x1="-195.58" y1="121.92" x2="-195.58" y2="127" width="0.1524" layer="91"/>
-<pinref part="U$2" gate="G$1" pin="CH2"/>
-<wire x1="-208.28" y1="152.4" x2="-208.28" y2="142.24" width="0.1524" layer="91"/>
-<wire x1="-195.58" y1="127" x2="-208.28" y2="142.24" width="0.1524" layer="91"/>
 <wire x1="-195.58" y1="121.92" x2="-182.88" y2="121.92" width="0.1524" layer="91"/>
-<junction x="-195.58" y="121.92"/>
 <label x="-193.04" y="121.92" size="1.778" layer="95"/>
 </segment>
@@
 <wire x1="-284.48" y1="129.54" x2="-302.26" y2="129.54" width="0.1524" layer="91"/>
 <junction x="-284.48" y="129.54"/>
-<junction x="-302.26" y="129.54"/>
 <label x="-302.26" y="137.16" size="1.778" layer="95"/>
-<pinref part="U$4" gate="G$1" pin="CH1"/>
-<wire x1="-274.32" y1="152.4" x2="-276.86" y2="149.86" width="0.1524" layer="91"/>
-<wire x1="-276.86" y1="149.86" x2="-299.72" y2="149.86" width="0.1524" layer="91"/>
-<wire x1="-299.72" y1="149.86" x2="-302.26" y2="147.32" width="0.1524" layer="91"/>
-<wire x1="-302.26" y1="147.32" x2="-302.26" y2="129.54" width="0.1524" layer="91"/>
 </segment>
 </net>
@@
 <wire x1="-241.3" y1="139.7" x2="-241.3" y2="129.54" width="0.1524" layer="91"/>
 <junction x="-241.3" y="129.54"/>
-<pinref part="U$2" gate="G$1" pin="CH1"/>
-<wire x1="-215.9" y1="152.4" x2="-223.52" y2="144.78" width="0.1524" layer="91"/>
-<wire x1="-223.52" y1="144.78" x2="-243.84" y2="144.78" width="0.1524" layer="91"/>
-<wire x1="-243.84" y1="144.78" x2="-243.84" y2="129.54" width="0.1524" layer="91"/>
-<junction x="-243.84" y="129.54"/>
 </segment>
 </net>
@@
 </segment>
 </net>
+<net name="N$2" class="0">
+<segment>
+<pinref part="R1" gate="G$1" pin="S"/>
+<pinref part="IC2" gate="A" pin="+IN"/>
+<wire x1="-154.94" y1="116.84" x2="-157.48" y2="116.84" width="0.1524" layer="91"/>
+</segment>
+</net>
